File: src/Mech Keyboard.kicad_pcb (KiCad board)
At the start: 2 copper layers, 360 x 139 mm, 169 parts

Commit message: Update to include new pcb
Parts:
- removed D86, D87: Diode, ScottoKeebs_Components:Diode_DO-35
- removed S86, S87: Keyswitch, ScottoKeebs_MX:MX_PCB_1.00u
- added D14: Diode, ScottoKeebs_Components:Diode_DO-35, F.Cu at (123.5, 58.3)
- added D15: Diode, ScottoKeebs_Components:Diode_DO-35, F.Cu at (142.5, 58.3)
- added D16: Diode, ScottoKeebs_Components:Diode_DO-35, F.Cu at (161.6, 58.3)
- added S14: Keyswitch, ScottoKeebs_MX:MX_PCB_1.00u, F.Cu at (114.1, 49.8)
- added S15: Keyswitch, ScottoKeebs_MX:MX_PCB_1.00u, F.Cu at (133.1, 49.8)
- added S16: Keyswitch, ScottoKeebs_MX:MX_PCB_1.00u, F.Cu at (152.2, 49.8)
- D1, D10, D11, D12, D13, D17, D18, D19, D2, D20, D21, D22, D23, D24, D25, D26, D27, D28, D29, D3, D30, D31, D32, D33, D34, D35, D36, D37, D38, D39, D4, D40, D41, D42, D43, D44, D45, D46, D47, D48, D49, D5, D50, D51, D52, D53, D54, D55, D56, D57, D58, D59, D6, D60, D61, D62, D63, D64, D65, D66, D67, D68, D69, D7, D70, D71, D72, D73, D74, D75, D76, D77, D78, D79, D8, D80, D81, D82, D83, D84, D85, D9: moved to F.Cu
- moved S79 278.1 mm to (306.9, 126.0)
- moved D79 277.9 mm to (316.3, 134.5)
- moved S80 240.0 mm to (330.8, 126.0)
- moved D80 239.8 mm to (340.2, 134.5)
- moved S74 230.5 mm to (423.6, 107.0)
- moved S78 230.5 mm to (235.5, 126.0)
- moved D74 230.3 mm to (433.0, 115.4)
- moved D78 230.3 mm to (244.9, 134.5)
- moved S28 216.2 mm to (404.6, 49.8)
- moved S29 216.2 mm to (423.6, 49.8)
- moved D29 216.0 mm to (433.0, 58.3)
- moved D28 216.0 mm to (414.0, 58.3)
- moved S30 206.7 mm to (442.7, 49.8)
- moved S46 206.7 mm to (423.6, 68.9)
- moved S45 206.7 mm to (404.6, 68.9)
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Connections:
- D31 pad 1: Row 1 -> Row 2
- D32 pad 1: Row 1 -> Row 2
- D33 pad 1: Row 1 -> Row 2
- D48 pad 1: Row 2 -> Row 3
- D49 pad 1: Row 2 -> Row 3
- D50 pad 1: Row 2 -> Row 3
- D61 pad 1: Row 3 -> Row 4
- D62 pad 1: Row 3 -> Row 4
- D63 pad 1: Row 3 -> Row 4
- D75 pad 1: Row 4 -> Row 5
- D76 pad 1: Row 4 -> Row 5
- S17 pad 1: Column 0 -> Column 3
- S18 pad 1: Column 1 -> Column 4
- S19 pad 1: Column 2 -> Column 5
- S20 pad 1: Column 3 -> Column 6
- S21 pad 1: Column 4 -> Column 7
- S22 pad 1: Column 5 -> Column 8
- S23 pad 1: Column 6 -> Column 9
- S24 pad 1: Column 7 -> Column 10
- S25 pad 1: Column 8 -> Column 11
- S26 pad 1: Column 9 -> Column 12
- S27 pad 1: Column 10 -> Column 13
- S28 pad 1: Column 11 -> Column 14
- S29 pad 1: Column 12 -> Column 15
- S30 pad 1: Column 13 -> Column 16
- S31 pad 1: Column 14 -> Column 0
- S32 pad 1: Column 15 -> Column 1
- S33 pad 1: Column 16 -> Column 2
- S34 pad 1: Column 0 -> Column 3
- S35 pad 1: Column 1 -> Column 4
- S36 pad 1: Column 2 -> Column 5
- S37 pad 1: Column 3 -> Column 6
- S38 pad 1: Column 4 -> Column 7
- S39 pad 1: Column 5 -> Column 8
- S40 pad 1: Column 6 -> Column 9
- S41 pad 1: Column 7 -> Column 10
- S42 pad 1: Column 8 -> Column 11
- S43 pad 1: Column 9 -> Column 12
- S44 pad 1: Column 10 -> Column 13
- S45 pad 1: Column 11 -> Column 14
- S46 pad 1: Column 12 -> Column 15
- S47 pad 1: Column 13 -> Column 16
- S48 pad 1: Column 14 -> Column 0
- S49 pad 1: Column 15 -> Column 1
- S50 pad 1: Column 16 -> Column 2
- S51 pad 1: Column 0 -> Column 3
- S52 pad 1: Column 1 -> Column 4
- S53 pad 1: Column 2 -> Column 5
- S54 pad 1: Column 3 -> Column 6
- S55 pad 1: Column 4 -> Column 7
- S56 pad 1: Column 5 -> Column 8
- S57 pad 1: Column 6 -> Column 9
- S58 pad 1: Column 7 -> Column 10
- S59 pad 1: Column 8 -> Column 11
- S60 pad 1: Column 9 -> Column 12
- S61 pad 1: Column 10 -> Column 0
- S62 pad 1: Column 11 -> Column 1
- S63 pad 1: Column 12 -> Column 2
- S64 pad 1: Column 0 -> Column 3
- S65 pad 1: Column 1 -> Column 4
- S66 pad 1: Column 2 -> Column 5
- S67 pad 1: Column 3 -> Column 6
- S68 pad 1: Column 4 -> Column 7
- S69 pad 1: Column 5 -> Column 8
- S70 pad 1: Column 6 -> Column 9
- S71 pad 1: Column 7 -> Column 10
- S72 pad 1: Column 8 -> Column 11
- S73 pad 1: Column 9 -> Column 12
- S74 pad 1: Column 10 -> Column 13
- S75 pad 1: Column 11 -> Column 1
- S76 pad 1: Column 12 -> Column 2
- S77 pad 1: Column 0 -> Column 3
- S78 pad 1: Column 1 -> Column 4
- S79 pad 1: Column 2 -> Column 5
- S80 pad 1: Column 3 -> Column 6
- S81 pad 1: Column 4 -> Column 7
- S82 pad 1: Column 5 -> Column 8
- S83 pad 1: Column 6 -> Column 9
- S84 pad 1: Column 7 -> Column 10
- S85 pad 1: Column 8 -> Column 11
Routing:
- net Column 10: track 736.9 -> 322.5 mm
- net Column 9: track 676.2 -> 347.0 mm
- net Column 8: track 682.5 -> 362.1 mm
- net Column 16: track 243.6 -> 62.7 mm
- net Net-(A1-GND-Pad13): track 119.2 -> 0.00 mm
- net Column 11: track 198.3 -> 300.6 mm
- net Column 13: track 91.8 -> 147.5 mm
- net Column 12: track 205.2 -> 157.8 mm
- net Column 4: track 433.9 -> 391.7 mm
- net Row 0: track 316.2 -> 284.0 mm
- net Column 0: track 467.7 -> 439.1 mm
- net Column 3: track 413.6 -> 388.8 mm
- net Row 1: track 351.6 -> 367.6 mm
- net Column 14: track 74.4 -> 60.0 mm
- net Net-(D15-A): track 0.00 -> 9.31 mm
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Other:
- board size 360 x 139 mm -> 350.5 x 129 mm
