File: src/Old/Mech Keyboard.kicad_sch (KiCad schematic)
At the start: 171 parts

Commit message: Update to include new pcb
Parts:
- removed D85: Diode, ScottoKeebs_Components:Diode_DO-35, symbol ScottoKeebs:Placeholder_Diode
- removed S85: Keyswitch, ScottoKeebs_MX:MX_PCB_1.00u, symbol ScottoKeebs:Placeholder_Keyswitch
- renumbered D14 to D17, D15 to D18, D16 to D19, D17 to D20, D18 to D21, D19 to D22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
Connections:
- net Column 0: now also S77.1
- net Column 13: no longer S77.1
- net Row 4: no longer D77.1 (K)
- net Row 5: now also D77.1 (K)
Other:
- moved on the sheet: D77, S77
